File: pcb.sch (EAGLE design)
At the start: 1 part, among them IC1 AT90S2333AA

Commit message: Adding memory
Parts:
- added IC2: (no value), memory-sram:MCM6290C
Changed lines of the file:
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@@
 <parts>
 <part name="IC1" library="atmel" deviceset="AT90S2333A" device="A"/>
+<part name="IC2" library="memory-sram" deviceset="MCM6290C" device=""/>
 </parts>
 <sheets>
@@
 <instances>
 <instance part="IC1" gate="G$1" x="40.64" y="50.8"/>
+<instance part="IC2" gate="G$1" x="88.9" y="58.42"/>
 </instances>
 <busses>
