File: USB to JTAG Programming Board.sch (EAGLE design)
At the start: 48 parts, among them CON1 UBC05V128-B0C04D, Q3 12M, U17 TPS62162DSGR, U5 ISO7240, U6 FT2232H, U7 ISO7231, U8 93LC56BT-I/OT

Commit message: Changed rev number and cleanup
Parts:
- U$1: value 1175-1733-ND -> IDC_BOX_HEADER_2X5_1.27MM; device MRDT-Connectors:1175-1733-ND -> MRDT-Connectors:IDC_BOX_HEADER_2X5_1.27MM
Changed lines of the file:
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@@
 <part name="GROUND" library="RF430FRL152H_EVM_a" deviceset="TESTPAD_TP" device="B1,27"/>
 <part name="3V3" library="RF430FRL152H_EVM_a" deviceset="TESTPAD_TP" device="B1,27"/>
-<part name="U$1" library="MRDT-Connectors" deviceset="1175-1733-ND" device=""/>
 <part name="U$2" library="MRDT-Signatures" deviceset="ANDREW_VAN_HORN_SIGNATURE" device=""/>
 <part name="LOGO1" library="MRDT-Hardware" deviceset="MRDT_LOGO" device=""/>
@@
 <part name="C2" library="eagle-ltspice" library_urn="urn:adsk.eagle:library:217" deviceset="C" device="C0603" package3d_urn="urn:adsk.eagle:package:13262/1" value="36p"/>
 <part name="C3" library="eagle-ltspice" library_urn="urn:adsk.eagle:library:217" deviceset="C" device="C0603" package3d_urn="urn:adsk.eagle:package:13262/1" value="36p"/>
+<part name="U$1" library="MRDT-Connectors" deviceset="IDC_BOX_HEADER_2X5_1.27MM" device=""/>
 </parts>
 <sheets>
@@
 <instance part="GROUND" gate="G$1" x="72.39" y="21.59" rot="R90"/>
 <instance part="3V3" gate="G$1" x="173.99" y="204.47"/>
-<instance part="U$1" gate="1" x="304.8" y="101.6"/>
 <instance part="U$2" gate="G$1" x="302.26" y="5.08"/>
 <instance part="LOGO1" gate="G$1" x="307.34" y="25.4"/>
@@
 <instance part="C2" gate="G$1" x="83.82" y="38.1" rot="R180"/>
 <instance part="C3" gate="G$1" x="93.98" y="38.1" rot="R180"/>
+<instance part="U$1" gate="1" x="309.88" y="101.6"/>
 </instances>
 <busses>
@@
 <wire x1="251.46" y1="96.52" x2="251.46" y2="53.34" width="0.1524" layer="91"/>
 <junction x="251.46" y="96.52"/>
-<wire x1="251.46" y1="106.68" x2="294.64" y2="106.68" width="0.1524" layer="91"/>
+<wire x1="251.46" y1="106.68" x2="304.8" y2="106.68" width="0.1524" layer="91"/>
 <pinref part="U$1" gate="1" pin="8-TDI"/>
-<wire x1="294.64" y1="106.68" x2="297.18" y2="106.68" width="0.1524" layer="91"/>
-<wire x1="304.8" y1="106.68" x2="297.18" y2="106.68" width="0.1524" layer="91"/>
 </segment>
 </net>
@@
 <wire x1="304.8" y1="104.14" x2="281.94" y2="104.14" width="0.1524" layer="91"/>
 <junction x="281.94" y="104.14"/>
+<pinref part="U$1" gate="1" pin="9-GND"/>
+<pinref part="U$1" gate="1" pin="7-RTCK"/>
+<pinref part="U$1" gate="1" pin="5-GND"/>
 <pinref part="U$1" gate="1" pin="3-GND"/>
-<pinref part="U$1" gate="1" pin="5-GND"/>
-<pinref part="U$1" gate="1" pin="7-RTCK"/>
-<pinref part="U$1" gate="1" pin="9-GND"/>
 </segment>
 <segment>
@@
 <wire x1="259.08" y1="96.52" x2="284.48" y2="96.52" width="0.1524" layer="91"/>
 <wire x1="284.48" y1="96.52" x2="284.48" y2="101.6" width="0.1524" layer="91"/>
-<wire x1="284.48" y1="101.6" x2="294.64" y2="101.6" width="0.1524" layer="91"/>
+<wire x1="284.48" y1="101.6" x2="304.8" y2="101.6" width="0.1524" layer="91"/>
 <pinref part="U$1" gate="1" pin="10-RST"/>
-<wire x1="294.64" y1="101.6" x2="297.18" y2="101.6" width="0.1524" layer="91"/>
-<wire x1="304.8" y1="101.6" x2="297.18" y2="101.6" width="0.1524" layer="91"/>
-</segment>
-</net>
+</segment>
+</net>
