File: 2015/Hardware/BMS_Rev3_logic.sch (EAGLE design)
At the start: 40 parts, among them Q1 2N7002PW, Q2 2N7002PW, Q9 MOSFET-NCHANNEL2N7002PW

Commit message: Working on BOM for Rev 3
Parts:
- L3: device rcl:L-USL4532C -> rcl:L-USL8530M
Changed lines of the file:
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@@
 <?xml version="1.0" encoding="utf-8"?>
 <!DOCTYPE eagle SYSTEM "eagle.dtd">
-<eagle version="6.5.0">
+<eagle version="7.0.0">
 <drawing>
 <settings>
@@
 <part name="GND1" library="SparkFun-Aesthetics" deviceset="GND" device=""/>
 <part name="C17" library="resistor" deviceset="C-US" device="C1206" value="47µF"/>
-<part name="L3" library="rcl" deviceset="L-US" device="L4532C" value="Fair-Rite 2773019447"/>
+<part name="L3" library="rcl" deviceset="L-US" device="L8530M" value="Fair-Rite 2773019447"/>
 <part name="C18" library="resistor" deviceset="C-US" device="C1206" value="47µF"/>
 <part name="GND10" library="SparkFun-Aesthetics" deviceset="GND" device=""/>
