File: hardware/failoverBoard.brd (EAGLE design)
At the start: 92.7 x 48.3 mm, 31 parts, among them J1 APP_2POS_CONFIG12V_HORIZ, U2 TINY45-20-DIP

Commit message: Add SL5 connectors for motors, passthrough serial data
Motors get independent control in normal mode, tank steer (left together, right together) in failover mode
Parts:
- removed IN1, IN2, OUT1, OUT2: SIERRAALTO.CONN.SUPPLEMENT_CONN_3MOLEX_0705550037, Rover_MC2:SIERRAALTO.CONN.SUPPLEMENT_MOLEX_0705550037_3
- removed R1: SELECT, rcl:M0805
- added C5: 0.1uF, SparkFun-Passives:0603-CAP
- added C6: 0.1uF, Rover_MC2:BOOST_CMP_0603-CAP
- added ML1IN, ML1OUT, ML2IN, ML2OUT, ML3IN, ML3OUT, MR1IN, MR1OUT, MR2IN, MR2OUT, MR3IN, MR3OUT: SL05VERT, MRDT-Connectors:MOLEX-70543-0004
- added MUX3: CD40257, ruark2:SOIC16
- added U1: OKI-78SR-3.3/1.5-W36HC, MRDT-ICs:OKI-78SR_HORIZ
Connections:
- removed net LOGIC_VCC: C2.1, C3.2, C4.1, MUX1.16, MUX2.16, U2.8
- removed net PWM_IN_1: IN1.2, MUX1.2
- removed net PWM_IN_2: IN2.2, MUX1.5
- removed net PWM_IN_VCC: IN1.3, IN2.3, IN3.3, IN4.3, IN5.3, IN6.3, IN7.3
- removed net PWM_OUT_1: MUX1.4, OUT1.2
- removed net PWM_OUT_2: MUX1.7, OUT2.2
- new net +3V3_LOGIC: C2.1, C3.2, C4.1, C5.1, C6.1, MUX1.16, MUX2.16, MUX3.16, U1.3, U2.8
- new net +5V: C1.+, IN3.2, IN4.2, IN5.2, IN6.2, IN7.2, OUT3.2, OUT4.2, OUT5.2, OUT6.2, OUT7.2, U$1.3
- new net ML1_PWM_IN: ML1IN.1, MUX3.2
- new net ML1_PWM_OUT: ML1OUT.1, MUX3.4
- new net ML2_PWM_IN: ML2IN.1, MUX3.5
- new net ML2_PWM_OUT: ML2OUT.1, MUX3.7
- new net ML3_PWM_IN: ML3IN.1, MUX3.11
- new net ML3_PWM_OUT: ML3OUT.1, MUX3.9
- new net MR1_PWM_IN: MR1IN.1, MUX3.14
- new net MR1_PWM_OUT: MR1OUT.1, MUX3.12
- new net MR2_PWM_IN: MR2IN.1, MUX1.2
- new net MR2_PWM_OUT: MR2OUT.1, MUX1.4
- new net MR3_PWM_IN: MR3IN.1, MUX1.5
- new net MR3_PWM_OUT: MR3OUT.1, MUX1.7
- new net N$10: ML1IN.2, ML1OUT.2
- new net N$11: MR1IN.2, MR1OUT.2
- new net N$12: MR1IN.4, MR1OUT.4
- new net N$13: MR1IN.5, MR1OUT.5
- new net N$14: MR2IN.4, MR2OUT.4
- new net N$15: MR2IN.5, MR2OUT.5
- new net N$16: MR3IN.4, MR3OUT.4
- new net N$17: MR3IN.5, MR3OUT.5
- new net N$18: MR3IN.2, MR3OUT.2
- new net N$19: MR2IN.2, MR2OUT.2
- new net N$2: ML1IN.4, ML1OUT.4
- new net N$3: ML2IN.4, ML2OUT.4
- new net N$4: ML2IN.5, ML2OUT.5
- new net N$5: ML1IN.5, ML1OUT.5
- new net N$6: ML3IN.4, ML3OUT.4
- new net N$7: ML3IN.5, ML3OUT.5
- new net N$8: ML3IN.2, ML3OUT.2
- new net N$9: ML2IN.2, ML2OUT.2
- net DL_CH1: now also MUX3.10, MUX3.3, MUX3.6; no longer MUX1.3
- net DL_CH2: now also MUX1.3, MUX3.13
- net GND: now also C5.2, C6.2, IN3.3, IN4.3, IN5.3, IN6.3, IN7.3, ML1IN.3, ML1OUT.3, ML2IN.3, ML2OUT.3, ML3IN.3, ML3OUT.3, MR1IN.3, MR1OUT.3, MR2IN.3, MR2OUT.3, MR3IN.3, MR3OUT.3, MUX3.8, OUT3.3, OUT4.3, OUT5.3, OUT6.3, OUT7.3, U1.2; no longer IN1.1, IN2.1, IN3.1, IN4.1, IN5.1, IN6.1, IN7.1, OUT1.1, OUT2.1, OUT3.1, OUT4.1, OUT5.1, OUT6.1, OUT7.1
- net MUX_ENABLE: now also MUX3.1
- net N$1: now also U1.1
- net PWM_IN_3: now also IN3.1; no longer IN3.2
- net PWM_IN_4: now also IN4.1; no longer IN4.2
- net PWM_IN_5: now also IN5.1; no longer IN5.2
- net PWM_IN_6: now also IN6.1; no longer IN6.2
- net PWM_IN_7: now also IN7.1; no longer IN7.2
- net PWM_OUT_3: now also OUT3.1; no longer OUT3.2
- net PWM_OUT_4: now also OUT4.1; no longer OUT4.2
- net PWM_OUT_5: now also OUT5.1; no longer OUT5.2
- net PWM_OUT_6: now also OUT6.1; no longer OUT6.2
- net PWM_OUT_7: now also OUT7.1; no longer OUT7.2
- net VCC: no longer C1.+, OUT1.3, OUT2.3, OUT3.3, OUT4.3, OUT5.3, OUT6.3, OUT7.3, U$1.3
Routing:
- net VCC: track 135.3 -> 17.8 mm
- net PWM_IN_VCC: track 91.1 -> 0.00 mm
- net +5V: track 0.00 -> 14.1 mm
- net LOGIC_VCC: track 8.63 -> 0.00 mm
- net +3V3_LOGIC: track 0.00 -> 8.63 mm
- net GND: track 16.0 -> 11.2 mm
