File: Science Board/Science-Board.brd (EAGLE design)
At the start: 104.1 x 55.9 mm, 66 parts, among them U3 SN74AHCT125

Commit message: Spectrometer Board: Removed unnecessary components from schematic and started board file from a clean slate.
Parts:
- removed C13: 4.7u, rcl:C0805
- removed C14: 10u, rcl:C0805
- removed CAROUSEL, FLAP: SERVOMOLEX_SL_THRU_HOLE, MRDT-Connectors:MOLEX_SL_03_TH
- removed GAS, HUMID, SOIL-MOIST, SOIL-TEMP, TEMP: SL03, MRDT-Connectors:MOLEX-70543-0002
- removed LIGHT, PRESSURE: SL04VERT, MRDT-Connectors:MOLEX-70543-0003
- removed R15, R2, R23, R27: 10k, rcl:R0805
- removed R22, R24, R28, R3: 19.3k, rcl:R0805
- removed U$2: LXDC2HN, MRDT-ICs:4-SMD
- removed U$4: KATIE-BRINKER, sig:KATIE-BRINKER-SIG
- removed U$8: TCA9517, MRDT-ICs:SOIC8
- removed U3: SN74AHCT125, MRDT-ICs:SOIC14
- moved R10 217.1 mm to (-128.3, 113.0), turned to 0 degrees
- moved R8 204.8 mm to (-121.9, 113.0), turned to 0 degrees
- moved SPEC-MOTOR 199.8 mm to (-106.7, 71.1), turned to 0 degrees
- moved C5 190.0 mm to (-90.2, 123.2)
- moved LASER 187.0 mm to (-123.2, 121.9)
- moved R6 186.9 mm to (-115.6, 113.0), turned to 0 degrees
- moved C12 180.6 mm to (-102.9, 113.0), turned to 0 degrees
- moved C10 180.5 mm to (-96.5, 113.0)
- moved R7 176.8 mm to (-100.3, 123.2), turned to 0 degrees
- moved R4 175.3 mm to (-109.2, 113.0), turned to 0 degrees
- moved R11 172.4 mm to (-74.9, 123.2), turned to 0 degrees
- moved C8 171.2 mm to (-95.2, 123.2)
- moved DIODE1 169.9 mm to (-119.4, 71.1)
- moved C11 166.7 mm to (-69.8, 123.2)
- moved U$7 165.4 mm to (-76.2, 113.0)
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Connections:
- removed net 3.3V: C14.1, LIGHT.1, LIGHT.4, SOIL-TEMP.2, U$2.P$3, U$8.1
- removed net N$11: CAROUSEL.3, U3.3
- removed net N$12: FLAP.3, U3.6
- removed net N$21: GAS.3, R15.2
- removed net N$22: HUMID.3, R27.2
- removed net N$6: R2.2, SOIL-MOIST.1
- removed net N$7: R23.2, TEMP.3
- removed net PRESSURE-SCL-5V: PRESSURE.1, U$8.7
- removed net PRESSURE-SDA-5V: PRESSURE.2, U$8.6
- net 5V-EXT: no longer C13.1, CAROUSEL.2, FLAP.2, GAS.1, HUMID.1, PRESSURE.4, SOIL-MOIST.2, TEMP.1, U$2.P$1, U$2.P$2, U$8.8, U3.14
- net GAS-A: no longer R15.1, R22.2
- net GND: no longer C13.2, C14.2, CAROUSEL.1, FLAP.1, GAS.2, HUMID.2, LIGHT.3, PRESSURE.3, R22.1, R24.1, R28.1, R3.1, SOIL-MOIST.3, SOIL-TEMP.3, TEMP.2, U$2.P$4, U$8.4, U3.1, U3.10, U3.13, U3.4, U3.7
- net HUMIDITY-A: no longer R27.1, R28.2
- net LEVEL-EN: no longer U$8.5
- net LIGHT-A: no longer LIGHT.2
- net PRESSURE-SCL-3V3: no longer U$8.2
- net PRESSURE-SDA-3V3: no longer U$8.3
- net SERVO-CAROUSEL: no longer U3.2
- net SERVO-FLAP: no longer U3.5
- net SOIL-MOISTURE: no longer R2.1, R3.2
- net SOIL-TEMP: no longer SOIL-TEMP.1
- net TEMP-A: no longer R23.1, R24.2
Routing:
- net 5V-EXT: track 164.0 -> 0.00 mm, vias 3 -> 0
- net 5V-INT: track 124.5 -> 0.00 mm, vias 6 -> 0
- net PRESSURE-SDA-3V3: track 86.4 -> 0.00 mm, vias 2 -> 0
- net PRESSURE-SCL-3V3: track 82.3 -> 0.00 mm, vias 2 -> 0
- net SOIL-TEMP: track 65.6 -> 0.00 mm, vias 2 -> 0
- net LIGHT-A: track 64.9 -> 0.00 mm, vias 1 -> 0
- net PHOTO-IN-2: track 59.9 -> 0.00 mm, vias 2 -> 0
- net GAS-A: track 47.2 -> 0.00 mm, vias 2 -> 0
- net 3.3V: track 40.1 -> 0.00 mm, vias 1 -> 0
- net TEMP-A: track 37.6 -> 0.00 mm
- net ACT-12V: track 36.1 -> 0.00 mm
- net N$12: track 35.7 -> 0.00 mm
- net LOGIC-12V: track 29.5 -> 0.00 mm
- net LASER-CTRL: track 27.7 -> 0.00 mm, vias 1 -> 0
- net PHOTO-IN: track 25.8 -> 0.00 mm
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- removed copper zone on layer 1, net GND
- removed copper zone on layer 16, net GND
Other:
- board size 104.1 x 55.9 mm -> 91.4 x 50.5 mm
- board text removed: "ACT"
- board text removed: "GND"
- board text removed: "LOG"
- board text removed: "Missouri S&T Mars Rover Design Team Science Board 2017 | Gryphon | Rev 2 Katie Brinker"
- board text removed: "sandstorm was here"
