File: GImbal Mastboard Rev-2/GImbal Mastboard Rev-2.kicad_pcb (KiCad board)
At the start: 2 copper layers, 59.8 x 55.1 mm, 31 parts, among them J1 Conn_01x03_Female, U1 TM4C123G, U2 OKI_12Vto3V3, U3 IMU-LSM90S1, U4 Raspberry_Pi_Header, U5 TIVA_C_TM4C123_Launchpad_Shie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, U6 JAG_ARM_Connector-10pin, U7 Molex_SL-4, U8 Molex_SL-3, Y1 16MHz

Commit message: Final touches before Bard Review
Other:
- net class Default: clearance 0.14224 -> 0.127
- rule trace_clearance: 0.14224 -> 0.127
Changed lines of the file:
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@@
     (links 118)
     (no_connects 2)
-    (area 118.917665 90.094999 178.898908 145.363001)
+    (area 118.18276 85.358102 180.59524 154.08086)
     (thickness 1.6)
     (drawings 17)
@@
     (user_trace_width 0.4064)
     (user_trace_width 0.508)
-    (trace_clearance 0.14224)
+    (trace_clearance 0.127)
     (zone_clearance 0.254)
     (zone_45_only yes)
@@
     (mod_text_size 1 1)
     (mod_text_width 0.15)
-    (pad_size 1.52 1.52)
-    (pad_drill 1)
+    (pad_size 3.45 3.45)
+    (pad_drill 3.45)
     (pad_to_mask_clearance 0.2)
     (aux_axis_origin 0 0)
@@
   (net 52 PD5)
   (net_class Default "This is the default net class."
-    (clearance 0.14224)
+    (clearance 0.127)
     (trace_width 0.25)
     (via_dia 0.5)
@@
     (fp_line (start 3.81 -1.27) (end 3.81 1.27) (layer F.SilkS) (width 0.15))
     (fp_line (start -3.81 1.27) (end -3.81 -1.27) (layer F.SilkS) (width 0.15))
-    (pad "" thru_hole circle (at -3.685 -8.64 180) (size 3.45 3.45) (drill 0.000254) (layers *.Cu *.Mask))
+    (pad "" np_thru_hole circle (at -3.685 -8.64 180) (size 3.45 3.45) (drill 3.45) (layers *.Cu *.Mask))
     (pad 1 thru_hole circle (at -2.54 0 180) (size 1.524 1.524) (drill 0.762) (layers *.Cu *.Mask)
       (net 17 PD7))
@@
       (net 22 PD6))
     (pad 3 thru_hole circle (at 2.54 0 180) (size 1.524 1.524) (drill 0.762) (layers *.Cu *.Mask))
-    (pad "" thru_hole circle (at 3.685 -8.64 180) (size 3.45 3.45) (drill 0.000254) (layers *.Cu *.Mask))
+    (pad "" np_thru_hole circle (at 3.685 -8.64 180) (size 3.45 3.45) (drill 3.45) (layers *.Cu *.Mask))
   )
   (module Socket_Strips:Socket_Strip_Straight_1x03_Pitch2.54mm (layer F.Cu)
@@
   (segment (start 150.942 111.252) (end 150.942 112.207) (width 0.254) (layer F.Cu) (net 4))
   (segment (start 150.942 112.207) (end 151.638 112.903) (width 0.254) (layer F.Cu) (net 4))
-  (segment (start 156.21 141.732) (end 156.972 141.732) (width 0.25) (layer B.Cu) (net 5) (status 400000))
+  (segment (start 156.21 141.732) (end 156.972 141.732) (width 0.25) (layer B.Cu) (net 5))
   (segment (start 173.8884 141.732) (end 156.972 141.732) (width 0.25) (layer B.Cu) (net 5))
-  (segment (start 173.8884 141.732) (end 174.498 141.1224) (width 0.25) (layer B.Cu) (net 5) (status 800000))
-  (segment (start 156.21 141.732) (end 155.9052 141.4272) (width 0.25) (layer B.Cu) (net 5) (status 400000))
-  (segment (start 156.486 141.996) (end 156.474 141.996) (width 0.25) (layer B.Cu) (net 5) (status C00000))
-  (segment (start 156.474 141.996) (end 155.9052 141.4272) (width 0.25) (layer B.Cu) (net 5) (status 400000))
+  (segment (start 173.8884 141.732) (end 174.498 141.1224) (width 0.25) (layer B.Cu) (net 5))
+  (segment (start 156.21 141.732) (end 155.9052 141.4272) (width 0.25) (layer B.Cu) (net 5))
+  (segment (start 156.486 141.996) (end 156.474 141.996) (width 0.25) (layer B.Cu) (net 5))
+  (segment (start 156.474 141.996) (end 155.9052 141.4272) (width 0.25) (layer B.Cu) (net 5))
   (segment (start 155.9052 141.4272) (end 155.575 141.097) (width 0.25) (layer B.Cu) (net 5))
   (segment (start 155.575 141.097) (end 155.1178 141.097) (width 0.25) (layer B.Cu) (net 5))
-  (segment (start 174.498 140.462) (end 174.498 141.1224) (width 0.25) (layer B.Cu) (net 5) (status C00000))
+  (segment (start 174.498 140.462) (end 174.498 141.1224) (width 0.25) (layer B.Cu) (net 5))
   (segment (start 174.8536 121.0564) (end 174.8536 128.27) (width 0.25) (layer B.Cu) (net 5))
   (segment (start 174.3952 120.598) (end 174.8536 121.0564) (width 0.254) (layer F.Cu) (net 5))
@@
   (segment (start 169.164 121.9835) (end 171.958 121.9835) (width 0.25) (layer F.Cu) (net 20))
   (segment (start 172.064282 122.089782) (end 172.085 122.1105) (width 0.25) (layer F.Cu) (net 20))
-  (segment (start 177.038 134.493) (end 177.0634 134.493) (width 0.25) (layer B.Cu) (net 21) (status C00000))
-  (segment (start 177.0634 134.493) (end 178.1048 135.5344) (width 0.25) (layer B.Cu) (net 21) (status 400000))
-  (segment (start 178.1048 139.3952) (end 177.038 140.462) (width 0.25) (layer B.Cu) (net 21) (status 800000))
+  (segment (start 177.038 134.493) (end 177.0634 134.493) (width 0.25) (layer B.Cu) (net 21))
+  (segment (start 177.0634 134.493) (end 178.1048 135.5344) (width 0.25) (layer B.Cu) (net 21))
+  (segment (start 178.1048 139.3952) (end 177.038 140.462) (width 0.25) (layer B.Cu) (net 21))
   (segment (start 178.1048 135.5344) (end 178.1048 139.3952) (width 0.25) (layer B.Cu) (net 21))
   (segment (start 177.038 134.493) (end 177.038 118.940956) (width 0.25) (layer B.Cu) (net 21))
