File: Gimbal Mastboard ESP/Gimbal Mastboard ESP.sch (KiCad schematic (older format))
At the start: 12 parts

Commit message: Generated Gerbs
Parts:
- added R2: 1M, Resistors_SMD:R_0603_HandSoldering, symbol R
- C1, C2, C3, C4: renamed from C?; footprint (none) -> Capacitors_SMD:C_0603_HandSoldering
- Conn1: renamed from Conn?; footprint (none) -> MRDT_Connectors:Anderson_2_Horisontal_Side_by_Side
- Conn2: renamed from Conn?; footprint (none) -> MRDT_Connectors:MOLEX_SL_4_Horizontal
- Conn3: renamed from Conn?; footprint (none) -> MRDT_Connectors:MOLEX_SL_3_Horizontal
- D1: renamed from D?; footprint (none) -> LEDs:LED_0603_HandSoldering
- R1: renamed from R?; footprint (none) -> Resistors_SMD:R_0603_HandSoldering
- U1: renamed from U?; footprint (none) -> MRDT_Shields:ESP_8266_Breakout_Small
- U2: renamed from U?; footprint (none) -> MRDT_Devices:OKI_Horisontal
- U3: renamed from U?; footprint (none) -> MRDT_Devices:IMU_LSM90S1
Connections:
- net +3V3: now also U3.12 (DENAG), U3.4 (SD0AG), U3.5 (SD0M), U3.6 (CSAG), U3.7 (CSM)
- net GND: now also R2.2
- net at U3.10 (INT1AG): now also U3.11 (INT2AG), U3.8 (DRDYM), U3.9 (INTM), R2.1
Other:
- note added: "Sets I2C Address"
- note added: "Sets I2C Mode"
- note added: "Unused Interupts"
- moved on the sheet: C1, C2, C3, C4, Conn1, D1, R1, U1
